File: 1.Hardware/1.FrontCar/1.MotherBoard/FrontCarMotherBoard.kicad_sch (KiCad schematic)
At the start: 44 parts

Commit message: 母板
Parts:
- removed Q?: S8050, Package_TO_SOT_THT:TO-92_Inline, symbol Transistor_BJT:S8050
- added D? (x2): 1N4148, Diode_SMD:D_SMA, symbol Simulation_SPICE:DIODE
- added D?: LED, symbol Device:LED
- added Q?: (no value), symbol Device:Q_NPN_BEC
- added Q?: (no value), Package_TO_SOT_SMD:SOT-23, symbol Device:Q_NPN_BEC
- added Q?: (no value), symbol ErBW_s:AO4803A
- added R? (x4): (no value), Resistor_SMD:R_1206_3216Metric_Pad1.30x1.75mm_HandSolder, symbol Device:R_Small
- U?: value (none) -> MT9V034; footprint (none) -> Connector_FFC-FPC:Hirose_FH12-18S-0.5SH_1x18-1MP_P0.50mm_Horizontal
Connections:
- net +3V3: now also R?.2
- net GND: now also Q?.2 (E)
- net GNDPWR: now also D?.1 (K), Q?.2 (E)
- net VBUS: now also Q?.1 (S2), R?.2
- net VCC: now also Q?.7 (D2_1), Q?.8 (D2_2)
- net at R?.2, R?.2: now also Q?.1 (B)
- net at R?.1: now also Q?.3 (C)
- new net: Q?.1 (B), R?.2, R?.2
- new net: D?.1 (A), Q?.2 (G2), Q?.3 (C), R?.1
- new net: D?.2 (A), R?.1
- new net: D?.2 (K), D?.2 (K)
- new net: D?.1 (A), R?.1
- no-connect marks 1 -> 5

Commit message: 更改电源开关模块
Parts:
- removed C?: 470uF, symbol Device:C_Polarized_Small_US
- removed D?: 1N4148, Diode_SMD:D_SMA, symbol Simulation_SPICE:DIODE
- removed SW?: SW_DPDT, symbol Switch:SW_DPDT_x2
- added C?: 470uF, symbol Device:C_Polarized_Small_US
- added SW?: (no value), symbol Switch:SW_Push
- Q?: value (none) -> FMMT619; footprint (none) -> Package_TO_SOT_SMD:SOT-23
- Q?: value (none) -> S8050
- Q?: value (none) -> AO4803A; footprint (none) -> SOIC127P600X175-8N
- R? (x3): value (none) -> 10K
- R?: value (none) -> 1K
Connections:
- net MOTORPWR is gone; now on net VCC: J?.1 (Pin_1)
- net GNDPWR: now also C?.2, SW?.1
- net VCC: now also C?.1
- net at D?.2 (K), D?.2 (K): now also SW?.2
- no-connect marks 5 -> 4
Other:
- moved on the sheet: R?

Commit message: 更改原理图为分层图框
Parts:
- removed C? (x8): 0.1uF, symbol Device:C_Small
- removed C? (x3): 10uF, symbol Device:C_Polarized_Small_US
- removed C? (x3): 22uF, symbol Device:C_Polarized_Small_US
- removed C?: 470uF, symbol Device:C_Polarized_Small_US
- removed D? (x4): LED, symbol Device:LED
- removed D? (x2): 1N4148, Diode_SMD:D_SMA, symbol Simulation_SPICE:DIODE
- removed IC?: SN74LVC244APW, SOP65P640X120-20N, symbol ErBW_s:SN74LVC244APW
- removed J?: PWR, Connector:VCC_CONN, symbol Connector_Generic:Conn_01x02
- removed J?: MOTOR, Connector:VCC_CONN, symbol Connector_Generic:Conn_01x02
- removed Q?: FMMT619, Package_TO_SOT_SMD:SOT-23, symbol Device:Q_NPN_BEC
- removed Q?: S8050, Package_TO_SOT_SMD:SOT-23, symbol Device:Q_NPN_BEC
- removed Q?: AO4803A, SOIC127P600X175-8N, symbol ErBW_s:AO4803A
- removed R? (x3): 5K1, symbol Device:R_Small
- removed R? (x3): 10K, Resistor_SMD:R_1206_3216Metric_Pad1.30x1.75mm_HandSolder, symbol Device:R_Small
- removed R? (x2): 1K, symbol Device:R_Small
- removed R?: 0R, Resistor_SMD:R_1206_3216Metric_Pad1.30x1.75mm_HandSolder, symbol Device:R_Small
- removed R?: 10R, symbol Device:R_Small
- removed R?: 1K, Resistor_SMD:R_1206_3216Metric_Pad1.30x1.75mm_HandSolder, symbol Device:R_Small
- removed R?: 10K, symbol Device:R_Small
- removed RV?: 3296W, symbol Device:R_Potentiometer
- removed SW?: (no value), symbol Switch:SW_Push
- removed SW?: SW_5DIR, ErBW_s:SW_5DIR, symbol ErBW_s:SW_5DIR
- removed SW?: SW_DIP_x04, symbol Switch:SW_DIP_x04
- removed TP?: 6V, TestPoint:TestPoint_Pad_D2.5mm, symbol Connector:TestPoint
- removed TP?: GND, TestPoint:TestPoint_Pad_2.5x2.5mm, symbol Connector:TestPoint
- removed TP?: 5V, TestPoint:TestPoint_Pad_D2.5mm, symbol Connector:TestPoint
- removed TP?: 3V3, TestPoint:TestPoint_Pad_D2.5mm, symbol Connector:TestPoint
- removed U?: LM2940S-5.0, symbol Regulator_Linear:LM2940S-5.0
- removed U?: IPS114, ErBW_s:IPS114, symbol ErBW_s:IPS114
- removed U?: LM1085-ADJ, symbol Regulator_Linear:LM1085-ADJ
- removed U?: MT9V034, Connector_FFC-FPC:Hirose_FH12-18S-0.5SH_1x18-1MP_P0.50mm_Horizontal, symbol ErBW_s:MT9V034
- removed U?: AMS1117-3.3, symbol Regulator_Linear:AMS1117-3.3
Connections:
- no-connect marks 4 -> 0
Other:
- added sheet Coreboard (Corboard.kicad_sch)
- added sheet Peripheral (Peripheral.kicad_sch)
- added sheet Ports (Ports.kicad_sch)
- added sheet Power (Power.kicad_sch)
- note added: "Copyright (c) 2022, ErBW_s All rights reserved."
