File: 1.Hardware/1.FrontCar/1.MotherBoard/Corboard.kicad_sch (KiCad schematic)
At the start: 1 part

Commit message: 增加版权信息
Other:
- note added: "Copyright (c) 2022, ErBW_s All rights reserved."
Changed lines of the file:
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@@
 (kicad_sch (version 20211123) (generator eeschema)
   (paper "A4")
+  (text "Copyright (c) 2022, ErBW_s\nAll rights reserved." (at 185.42 180.34 0)
+    (effects (font (size 4.318 4.318)) (justify left bottom))
+  )
   (symbol (lib_id "Device:Fuse_Small") (at 115.57 73.66 0) (unit 1)
     (in_bom yes) (on_board yes) (fields_autoplaced)
