File: 1.Hardware/1.FrontCar/1.MotherBoard/Peripheral.kicad_sch (KiCad schematic)
At the start: 11 parts

Commit message: 增加版权信息
Other:
- note added: "Copyright (c) 2022, ErBW_s All rights reserved."
Changed lines of the file:
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@@
     (stroke (width 0) (type default) (color 0 0 0 0))
+  )
+  (text "Copyright (c) 2022, ErBW_s\nAll rights reserved." (at 186.69 180.34 0)
+    (effects (font (size 4.318 4.318)) (justify left bottom))
   )
   (label "LEDK" (at 111.76 58.42 0)
