File: 1.Hardware/1.FrontCar/1.MotherBoard/Power.kicad_sch (KiCad schematic)
At the start: 39 parts

Commit message: 增加版权信息
Other:
- note added: "Copyright (c) 2022, ErBW_s All rights reserved."
Changed lines of the file:
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@@
     (stroke (width 0) (type default) (color 0 0 0 0))
+  )
+  (text "Copyright (c) 2022, ErBW_s\nAll rights reserved." (at 186.69 180.34 0)
+    (effects (font (size 4.318 4.318)) (justify left bottom))
   )
   (symbol (lib_id "Device:C_Small") (at 160.02 36.83 0) (unit 1)
