File: 1.Hardware/1.FrontCar/1.Coreboard/MM32F5_CoreBoard.kicad_sch (KiCad schematic)
At the start: 21 parts

Commit message: Update coreboard sch
Parts:
- added C? (x3): (no value), symbol Device:C_Small
- added C?: 0.1uF, symbol Device:C_Small
- added R?: 120R, symbol Device:R_Small
- added R?: 4.7K, symbol Device:R_Small
- added R? (x2): (no value), symbol Device:R_Small
- added U?: (no value), symbol Interface_CAN_LIN:SN65HVD232
- added U?: SN65HVD232, Package_SO:SOIC-8_3.9x4.9mm_P1.27mm, symbol Interface_CAN_LIN:SN65HVD232
- added U?: (no value), symbol Sensor_Motion:MPU-6050
Connections:
- net +3.3VA: now also C?.2, C?.2, R?.1, R?.1, U?.13 (VDD), U?.3 (VCC), U?.3 (VCC), U?.8 (VDDIO)
- net GND: now also C?.1, C?.1, C?.2, C?.2, U?.1 (CLKIN), U?.11 (FSYNC), U?.18 (GND), U?.2 (GND), U?.2 (GND), U?.9 (AD0)
- new net: C?.1, U?.10 (REGOUT)
- new net: C?.1, U?.20 (CPOUT)
- new net CAN1_D: U?.1 (D)
- new net CAN1_H: R?.1, U?.7 (CANH)
- new net CAN1_L: R?.2, U?.6 (CANL)
- new net CAN1_R: U?.4 (R)
- new net CAN2_D: U?.1 (D)
- new net CAN2_H: R?.1, U?.7 (CANH)
- new net CAN2_L: R?.2, U?.6 (CANL)
- new net CAN2_R: U?.4 (R)
- new net IMU_SCL: R?.2, U?.23 (SCL)
- new net IMU_SDA: R?.2, U?.24 (SDA)
- no-connect marks 0 -> 3

Commit message: 核心板
Parts:
- added C? (x12): 100nF, symbol Device:C_Small
- added C? (x6): (no value), symbol Device:C_Small
- added C? (x2): 0.1uF, symbol Device:C_Small
- added D?: (no value), symbol Diode:1N5819WS
- added D?: (no value), symbol Device:LED_Small
- added F?: (no value), symbol Device:Fuse_Small
- added R?: (no value), symbol Device:R_Small
- added U?: (no value), symbol ErBW_s:RT9013-33GB
- added U?: CH340E, Package_SO:MSOP-10_3x3mm_P0.5mm, symbol Interface_USB:CH340E
- Q?: value S8050 -> (none)
Connections:
- net +3V3 is gone; now on net +3.3VA: C?.1, C?.1, R?.1, U?.10 (VCC), U?.12 (LEDA)
- net BLK is gone; now on net IPS_BLK: R?.1
- net +3.3VA: now also C?.1, C?.1, C?.2, C?.2, C?.2, C?.2, C?.2, C?.2, C?.2, C?.2, C?.2, C?.2, C?.2, C?.2, R?.1, U?.5 (VOUT)
- net CAN1_D: now also U?.140 (PB9)
- net CAN1_R: now also U?.139 (PB8)
- net CAN2_D: now also U?.74 (PB13)
- net CAN2_R: now also U?.73 (PB12)
- net GND: now also J?.A1 (GND), J?.A12 (GND), J?.B1 (GND), J?.B12 (GND), J?.S1 (SHIELD), R?.2, R?.2, C?.1, C?.1, C?.1, C?.1, C?.1, C?.1, C?.1, C?.1, C?.1, C?.1, C?.1, C?.1, C?.1, C?.1, C?.1, C?.1, C?.1, C?.2, C?.2, C?.2, D?.1 (K), U?.2 (GND), U?.3 (GND)
- net IMU_SCL: now also U?.96 (PC6)
- net IMU_SDA: now also U?.97 (PC7)
- net IPS_SCL: now reaches U?.118 (PD4)
- net IPS_SCL: now also U?.4 (SCL)
- net IPS_DC: now reaches U?.119 (PD5)
- net IPS_DC: now also U?.5 (RS)
- net IPS_SDA: now reaches U?.122 (PD6)
- net IPS_SDA: now also U?.3 (SDA)
- net IPS_CS: now reaches U?.123 (PD7)
- net IPS_CS: now also U?.7 (CS)
- net UART1_TX: now reaches U?.136 (PB6)
- net UART1_TX: now also U?.9 (RXD)
- net UART1_RX: now reaches U?.137 (PB7)
- net UART1_RX: now also U?.8 (TXD)
- net IPS_RES: now reaches U?.85 (PD14)
- net IPS_RES: now also U?.6 (RES)
- net IPS_BLK: now reaches U?.86 (PD15)
- net +5V: now reaches J?.A4 (VBUS), J?.A9 (VBUS), J?.B4 (VBUS), J?.B9 (VBUS)
- net +5V: now also C?.2, D?.2 (A)
- net at J?.A6 (D+): now also J?.B6 (D+), U?.1 (UD+)
- net at J?.A7 (D-): now also J?.B7 (D-), U?.2 (UD-)
- new net: D?.1 (K), F?.1
- new net: D?.2 (A), R?.2
- new net: C?.1, U?.4 (NC)
- new net: C?.2, U?.10 (V3)
- new net +5VA: C?.2, C?.2, C?.2, F?.2, U?.1 (VIN), U?.3 (EN), U?.7 (VCC)
- no-connect marks 3 -> 8
Other:
- note added: "CAN"
- note added: "Copyright (c) 2022, ErBW_s All rights reserved."
- note added: "IPS114"
- note added: "MPU6050"
- note added: "PWR & FILTER"
- note added: "USB TO TTL"
- note added: "XTAL & RST"
- moved on the sheet: C?, J?, Q?, R?, SW?, U?, Y?

Commit message: 继续完善
Parts:
- removed C?: 100nF, symbol Device:C_Small
- added C?: (no value), symbol Device:C_Small
- added J? (x2): (no value), symbol Connector_Generic:Conn_02x25_Odd_Even
- added J?: (no value), symbol Connector_Generic_MountingPin:Conn_01x04_MountingPin
- added R?: 10K, symbol Device:R_Small
- C? (x3): value (none) -> 100nF
- C? (x2): value (none) -> 10nF
- C? (x2): value (none) -> 10uF
- C?: value (none) -> 18pF
- C?: value (none) -> 2.2nF
- C?: value (none) -> 0.1uF
- D?: value (none) -> 1N5819; footprint (none) -> Diode_SMD:D_SOD-323
- D?: value (none) -> GREEN
- F?: value (none) -> 350mA
- J?: value (none) -> USB_C_Receptacle_USB2.0
- Q?: value (none) -> FMMT619
- R?: value (none) -> 10K
- R? (x2): value (none) -> 5.1K
- R? (x2): value (none) -> 4.7K
- R?: value (none) -> 120R
- R?: value (none) -> 510R
- SW?: value (none) -> 3x4
- U?: footprint (none) -> Package_QFP:LQFP-144_20x20mm_P0.5mm
- U?: value (none) -> RT9013-33GB; footprint (none) -> Package_TO_SOT_SMD:SOT-23-5
- U?: value (none) -> SN65HVD232; footprint (none) -> Package_SO:SOIC-8_3.9x4.9mm_P1.27mm
- U?: value (none) -> MPU-6050; footprint (none) -> Sensor_Motion:InvenSense_QFN-24_4x4mm_P0.5mm
Connections:
- net +3.3VA: now also U?.108 (VDD), U?.121 (VDD), U?.131 (VDD), U?.144 (VDD), U?.17 (VDD), U?.32 (VREF+), U?.33 (VDDA), U?.39 (VDD), U?.52 (VDD), U?.6 (VBAT), U?.62 (VDD), U?.72 (VDD), U?.84 (VDD), U?.95 (VDD), C?.2, J?.1 (Pin_1)
- net GND: now also U?.107 (VSS), U?.120 (VSS), U?.130 (VSS), U?.143 (VSS), U?.16 (VSS), U?.30 (VSSA), U?.31 (VREF-), U?.38 (VSS), U?.51 (VSS), U?.61 (VSS), U?.71 (VSS), U?.83 (VSS), U?.94 (VSS), C?.1, J?.4 (Pin_4), J?.MP (MountPin), R?.1
- net SWDIO: now reaches U?.105 (SWDIO)
- net SWDIO: now also J?.2 (Pin_2)
- net SWCLK: now reaches U?.109 (SWCLK)
- net SWCLK: now also J?.3 (Pin_3)
- net at U?.138 (PH3-BOOT0): now also R?.2
Other:
- moved on the sheet: C?

Commit message: 更新
Parts:
- gave numbers to parts that had none: 1
Connections:
- net CAM_RXD: now reaches U?.113 (PC12)
- net CAM_TXD: now reaches U?.116 (PD2)
- net CAM_D0: now reaches U?.56 (PG0)
- net CAM_D1: now reaches U?.57 (PG1)
- net CAM_PLCK: now reaches U?.58 (PE7)
- net CAM_VSYNC: now reaches U?.59 (PE8)
- net CAM_D2: now reaches U?.87 (PG2)
- net CAM_D3: now reaches U?.88 (PG3)
- net CAM_D4: now reaches U?.89 (PG4)
- net CAM_D5: now reaches U?.90 (PG5)
- net CAM_D6: now reaches U?.91 (PG6)
- net CAM_D7: now reaches U?.92 (PG7)
Changed lines of the file:
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@@
     (stroke (width 0) (type default) (color 0 0 0 0))
   )
+  (wire (pts (xy 279.4 148.59) (xy 266.7 148.59))
+    (stroke (width 0) (type default) (color 0 0 0 0))
+  )
   (wire (pts (xy 375.92 186.69) (xy 382.27 186.69))
     (stroke (width 0) (type default) (color 0 0 0 0))
@@
     (stroke (width 0) (type default) (color 0 0 0 0))
   )
+  (wire (pts (xy 223.52 214.63) (xy 223.52 201.93))
+    (stroke (width 0) (type default) (color 0 0 0 0))
+  )
   (wire (pts (xy 336.55 63.5) (xy 341.63 63.5))
     (stroke (width 0) (type default) (color 0 0 0 0))
   )
+  (wire (pts (xy 238.76 85.09) (xy 238.76 97.79))
+    (stroke (width 0) (type default) (color 0 0 0 0))
+  )
   (wire (pts (xy 44.45 146.05) (xy 40.64 146.05))
     (stroke (width 0) (type default) (color 0 0 0 0))
@@
     (stroke (width 0) (type default) (color 0 0 0 0))
   )
+  (wire (pts (xy 220.98 214.63) (xy 220.98 201.93))
+    (stroke (width 0) (type default) (color 0 0 0 0))
+  )
   (wire (pts (xy 341.63 63.5) (xy 349.25 63.5))
     (stroke (width 0) (type default) (color 0 0 0 0))
@@
     (stroke (width 0) (type default) (color 0 0 0 0))
   )
+  (wire (pts (xy 279.4 153.67) (xy 266.7 153.67))
+    (stroke (width 0) (type default) (color 0 0 0 0))
+  )
   (wire (pts (xy 60.96 71.12) (xy 60.96 73.66))
     (stroke (width 0) (type default) (color 0 0 0 0))
@@
     (stroke (width 0) (type default) (color 0 0 0 0))
   )
+  (wire (pts (xy 246.38 85.09) (xy 246.38 97.79))
+    (stroke (width 0) (type default) (color 0 0 0 0))
+  )
   (wire (pts (xy 328.93 186.69) (xy 332.74 186.69))
     (stroke (width 0) (type default) (color 0 0 0 0))
@@
     (stroke (width 0) (type default) (color 0 0 0 0))
   )
+  (wire (pts (xy 279.4 158.75) (xy 266.7 158.75))
+    (stroke (width 0) (type default) (color 0 0 0 0))
+  )
   (wire (pts (xy 347.98 240.03) (xy 347.98 237.49))
     (stroke (width 0) (type default) (color 0 0 0 0))
@@
     (stroke (width 0) (type default) (color 0 0 0 0))
   )
+  (wire (pts (xy 279.4 146.05) (xy 266.7 146.05))
+    (stroke (width 0) (type default) (color 0 0 0 0))
+  )
+  (wire (pts (xy 218.44 214.63) (xy 218.44 201.93))
+    (stroke (width 0) (type default) (color 0 0 0 0))
+  )
   (wire (pts (xy 52.07 39.37) (xy 52.07 40.64))
     (stroke (width 0) (type default) (color 0 0 0 0))
@@
     (stroke (width 0) (type default) (color 0 0 0 0))
   )
+  (wire (pts (xy 279.4 151.13) (xy 266.7 151.13))
+    (stroke (width 0) (type default) (color 0 0 0 0))
+  )
   (polyline (pts (xy 20.32 165.1) (xy 20.32 124.46))
     (stroke (width 0) (type default) (color 0 0 0 0))
@@
     (stroke (width 0) (type default) (color 0 0 0 0))
   )
+  (wire (pts (xy 279.4 156.21) (xy 266.7 156.21))
+    (stroke (width 0) (type default) (color 0 0 0 0))
+  )
   (wire (pts (xy 266.7 194.31) (xy 279.4 194.31))
     (stroke (width 0) (type default) (color 0 0 0 0))
@@
     (stroke (width 0) (type default) (color 0 0 0 0))
   )
+  (wire (pts (xy 215.9 214.63) (xy 215.9 201.93))
+    (stroke (width 0) (type default) (color 0 0 0 0))
+  )
   (wire (pts (xy 226.06 95.25) (xy 226.06 97.79))
     (stroke (width 0) (type default) (color 0 0 0 0))
@@
     (effects (font (size 1.27 1.27)) (justify left bottom))
   )
+  (label "CAM_D7" (at 279.4 146.05 180)
+    (effects (font (size 1.27 1.27)) (justify right bottom))
+  )
   (label "OSC32_IN" (at 87.63 138.43 0)
     (effects (font (size 1.27 1.27)) (justify left bottom))
@@
     (effects (font (size 1.27 1.27)) (justify right bottom))
   )
+  (label "CAM_D4" (at 279.4 153.67 180)
+    (effects (font (size 1.27 1.27)) (justify right bottom))
+  )
   (label "SWCLK" (at 340.36 232.41 0)
     (effects (font (size 1.27 1.27)) (justify left bottom))
@@
     (effects (font (size 1.27 1.27)) (justify left bottom))
   )
+  (label "CAM_VSYNC" (at 223.52 214.63 90)
+    (effects (font (size 1.27 1.27)) (justify left bottom))
+  )
   (label "CAN1_H" (at 332.74 186.69 0)
     (effects (font (size 1.27 1.27)) (justify left bottom))
@@
     (effects (font (size 1.27 1.27)) (justify right bottom))
   )
+  (label "CAM_TXD" (at 238.76 85.09 270)
+    (effects (font (size 1.27 1.27)) (justify right bottom))
+  )
   (label "IPS_SDA" (at 223.52 85.09 270)
     (effects (font (size 1.27 1.27)) (justify right bottom))
@@
     (effects (font (size 1.27 1.27)) (justify left bottom))
   )
+  (label "CAM_RXD" (at 246.38 85.09 270)
+    (effects (font (size 1.27 1.27)) (justify right bottom))
+  )
   (label "IPS_RES" (at 350.52 41.91 0)
     (effects (font (size 1.27 1.27)) (justify left bottom))
   )
+  (label "CAM_D1" (at 218.44 214.63 90)
+    (effects (font (size 1.27 1.27)) (justify left bottom))
+  )
   (label "IPS_RES" (at 279.4 163.83 180)
     (effects (font (size 1.27 1.27)) (justify right bottom))
@@
     (effects (font (size 1.27 1.27)) (justify right bottom))
   )
+  (label "CAM_D2" (at 279.4 158.75 180)
+    (effects (font (size 1.27 1.27)) (justify right bottom))
+  )
   (label "IMU_SDA" (at 317.5 118.11 0)
     (effects (font (size 1.27 1.27)) (justify left bottom))
@@
     (effects (font (size 1.27 1.27)) (justify left bottom))
   )
+  (label "CAM_PLCK" (at 220.98 214.63 90)
+    (effects (font (size 1.27 1.27)) (justify left bottom))
+  )
   (label "RST" (at 106.68 144.78 0)
     (effects (font (size 1.27 1.27)) (justify left bottom))
@@
     (effects (font (size 1.27 1.27)) (justify left bottom))
   )
+  (label "CAM_D3" (at 279.4 156.21 180)
+    (effects (font (size 1.27 1.27)) (justify right bottom))
+  )
+  (label "CAM_D6" (at 279.4 148.59 180)
+    (effects (font (size 1.27 1.27)) (justify right bottom))
+  )
   (label "IPS_SCL" (at 350.52 36.83 0)
     (effects (font (size 1.27 1.27)) (justify left bottom))
@@
     (effects (font (size 1.27 1.27)) (justify left bottom))
   )
+  (label "CAM_D5" (at 279.4 151.13 180)
+    (effects (font (size 1.27 1.27)) (justify right bottom))
+  )
   (label "UART1_TX" (at 187.96 85.09 270)
     (effects (font (size 1.27 1.27)) (justify right bottom))
   )
+  (label "CAM_D0" (at 215.9 214.63 90)
+    (effects (font (size 1.27 1.27)) (justify left bottom))
+  )
   (symbol (lib_id "power:GND") (at 54.61 45.72 0) (unit 1)
     (in_bom yes) (on_board yes) (fields_autoplaced)
@@
   (symbol (lib_id "ErBW_s:IPS114") (at 370.84 44.45 0) (unit 1)
     (in_bom yes) (on_board yes) (fields_autoplaced)
-    (property "Reference" "U?" (id 0) (at 376.682 43.6153 0)
+    (property "Reference" "J?" (id 0) (at 376.682 43.6153 0)
       (effects (font (size 1.27 1.27)) (justify left))
     )
@@
       (reference "J?") (unit 1) (value "SH1.0_4P") (footprint "Connector_JST:JST_SH_SM04B-SRSS-TB_1x04-1MP_P1.00mm_Horizontal")
     )
+    (path "/dc48cb12-ea35-4f7d-a2e1-838d59de09d2"
+      (reference "J?") (unit 1) (value "IPS114") (footprint "ErBW_s:IPS114")
+    )
     (path "/57bb90af-663a-41d6-b400-0d4f24259321"
       (reference "Q?") (unit 1) (value "FMMT619") (footprint "Package_TO_SOT_SMD:SOT-23")
@@
       (reference "U?") (unit 1) (value "MPU-6050") (footprint "Sensor_Motion:InvenSense_QFN-24_4x4mm_P0.5mm")
     )
-    (path "/dc48cb12-ea35-4f7d-a2e1-838d59de09d2"
-      (reference "U?") (unit 1) (value "IPS114") (footprint "ErBW_s:IPS114")
-    )
     (path "/53b13b37-e8f3-459b-8efe-4bb4b0a93f96"

Commit message: 引出全部引脚
Connections:
- net IMU_SCL: now also U?.26 (PC0); no longer U?.96 (PC6)
- net IMU_SDA: now also U?.27 (PC1); no longer U?.97 (PC7)
- net PE2: now reaches U?.1 (PE2)
- net PF0: now reaches U?.10 (PF0)
- net PA8: now reaches U?.100 (PA8)
- net PA9: now reaches U?.101 (PA9)
- net PA10: now reaches U?.102 (PA10)
- net PA11: now reaches U?.103 (PA11)
- net PA12: now reaches U?.104 (PA12)
- net PH2: now reaches U?.106 (PH2)
- net PF1: now reaches U?.11 (PF1)
- net SERVO: now reaches U?.110 (PA15)
- net PC10: now reaches U?.111 (PC10)
- net PC11: now reaches U?.112 (PC11)
- net PD0: now reaches U?.114 (PD0)
- net PD1: now reaches U?.115 (PD1)
- net PD3: now reaches U?.117 (PD3)
- net PF2: now reaches U?.12 (PF2)
- net PG9: now reaches U?.124 (PG9)
- net PG10: now reaches U?.125 (PG10)
- net PG11: now reaches U?.126 (PG11)
- net PG12: now reaches U?.127 (PG12)
- net PG13: now reaches U?.128 (PG13)
- net PG14: now reaches U?.129 (PG14)
- net PF3: now reaches U?.13 (PF3)
- net PG15: now reaches U?.132 (PG15)
- net PB3: now reaches U?.133 (PB3)
- net 1LSB: now reaches U?.134 (PB4)
- net 1DIR: now reaches U?.135 (PB5)
- net 1DIR: now also U?.34 (PA0)
- net PF4: now reaches U?.14 (PF4)
- net PE0: now reaches U?.141 (PE0)
- net PE1: now reaches U?.142 (PE1)
- net PF5: now reaches U?.15 (PF5)
- net PF6: now reaches U?.18 (PF6)
- net PF7: now reaches U?.19 (PF7)
- net PE3: now reaches U?.2 (PE3)
- net PF8: now reaches U?.20 (PF8)
- net PF9: now reaches U?.21 (PF9)
- net PF10: now reaches U?.22 (PF10)
- net ADC_VBAT: now reaches U?.28 (PC2)
- net ADC_DIS: now reaches U?.29 (PC3)
- net PE4: now reaches U?.3 (PE4)
- net 1PWM: now reaches U?.35 (PA1)
- net 2DIR: now reaches U?.36 (PA2)
- net 2DIR: now also U?.82 (PD13)
- net 2PWM: now reaches U?.37 (PA3)
- net TOF_SCL: now reaches U?.4 (PE5)
- net ELEMAG1: now reaches U?.40 (PA4)
- net ELEMAG2: now reaches U?.41 (PA5)
- net ELEMAG3: now reaches U?.42 (PA6)
- net ELEMAG4: now reaches U?.43 (PA7)
- net ELEMAG5: now reaches U?.44 (PC4)
- net PC5: now reaches U?.45 (PC5)
- net PB0: now reaches U?.46 (PB0)
- net PB1: now reaches U?.47 (PB1)
- net PB2-BOOT1: now reaches U?.48 (PB2-BOOT1)
- net PF11: now reaches U?.49 (PF11)
- net TOF_SDA: now reaches U?.5 (PE6)
- net PF12: now reaches U?.50 (PF12)
- net PF13: now reaches U?.53 (PF13)
- net PF14: now reaches U?.54 (PF14)
- net PF15: now reaches U?.55 (PF15)
- net PE9: now reaches U?.60 (PE9)
- net PE10: now reaches U?.63 (PE10)
- net MAPLE_CS: now reaches U?.64 (PE11)
- net MAPLE_CLK: now reaches U?.65 (PE12)
- net MAPLE_MISO: now reaches U?.66 (PE13)
- net MAPLE_MOSI: now reaches U?.67 (PE14)
- net PE15: now reaches U?.68 (PE15)
- net PB10: now reaches U?.69 (PB10)
- net PC13: now reaches U?.7 (PC13)
- net PB11: now reaches U?.70 (PB11)
- net PB14: now reaches U?.75 (PB14)
- net PB15: now reaches U?.76 (PB15)
- net PD8: now reaches U?.77 (PD8)
- net PD9: now reaches U?.78 (PD9)
- net PD10: now reaches U?.79 (PD10)
- net PD11: now reaches U?.80 (PD11)
- net 2LSB: now reaches U?.81 (PD12)
- net PG8: now reaches U?.93 (PG8)
- net PC8: now reaches U?.98 (PC8)
- net PC9: now reaches U?.99 (PC9)
- new net ENCODER_A: U?.96 (PC6)
- new net ENCODER_B: U?.97 (PC7)
Other:
- note added: "FILTER"
- note added: "PWR"
- note added: "SWD"
- note removed: "PWR & FILTER"
- moved on the sheet: C?, J?, R?, SW?, U?, Y?

Commit message: 胡言乱语ing
Parts:
- removed F?: 350mA, symbol Device:Fuse_Small
- C?: value (none) -> 100nF
- D?: value 1N5819 -> (none); footprint Diode_SMD:D_SOD-323 -> (none)
- J? (x2): value (none) -> BTB_02x25
- J?: value (none) -> SH1.0_4P; footprint (none) -> Connector_JST:JST_SH_SM04B-SRSS-TB_1x04-1MP_P1.00mm_Horizontal
- U?: value (none) -> MM32F5277E9P
- Y?: value (none) -> 32.768KHz; footprint (none) -> ErBW_s:Crystal_SMD_3215_FC-135_2P
- Y?: value (none) -> 8MHz; footprint (none) -> ErBW_s:Crystal_SMD_3213_3P
Connections:
- net +5V: now also D?.1 (K); no longer D?.2 (A)
- net +5VA: now also D?.2 (A)
Other:
- moved on the sheet: C?
