File: 1.Hardware/1.FrontCar/1.Coreboard/_autosave-MM32F5_CoreBoard.kicad_sch (KiCad schematic)
At the start: 61 parts

Commit message: 增加封装
Parts:
- added R?: 0R, ErBW_s:R_0402, symbol Device:R_Small
- added R?: (no value), ErBW_s:R_0402, symbol Device:R_Small
Connections:
- net +3.3VA: now also R?.1; no longer C?.1, C?.1, C?.1, C?.1, C?.2, C?.2, C?.2, C?.2, C?.2, C?.2, C?.2, C?.2, C?.2, C?.2, C?.2, C?.2, C?.2, J?.1 (Pin_1), J?.10 (VCC), J?.12 (LEDA), R?.1, R?.1, R?.1, R?.1, R?.1, U?.108 (VDD), U?.121 (VDD), U?.13 (VDD), U?.131 (VDD), U?.144 (VDD), U?.17 (VDD), U?.3 (VCC), U?.3 (VCC), U?.39 (VDD), U?.5 (VOUT), U?.52 (VDD), U?.6 (VBAT), U?.62 (VDD), U?.72 (VDD), U?.8 (VDDIO), U?.84 (VDD), U?.95 (VDD)
- net GND: now also R?.2; no longer C?.1, U?.30 (VSSA), U?.31 (VREF-)
- new net +3.3V: C?.1, C?.1, C?.1, C?.1, C?.2, C?.2, C?.2, C?.2, C?.2, C?.2, C?.2, C?.2, C?.2, C?.2, C?.2, C?.2, C?.2, J?.1 (Pin_1), J?.10 (VCC), J?.12 (LEDA), R?.1, R?.1, R?.1, R?.1, R?.1, R?.2, U?.108 (VDD), U?.121 (VDD), U?.13 (VDD), U?.131 (VDD), U?.144 (VDD), U?.17 (VDD), U?.3 (VCC), U?.3 (VCC), U?.39 (VDD), U?.5 (VOUT), U?.52 (VDD), U?.6 (VBAT), U?.62 (VDD), U?.72 (VDD), U?.8 (VDDIO), U?.84 (VDD), U?.95 (VDD)
- new net GNDA: C?.1, R?.1, U?.30 (VSSA), U?.31 (VREF-)
Other:
- moved on the sheet: C?, D?, R?, U?
