File: 1.Hardware/1.FrontCar/1.CoreBoard/MM32F5_CoreBoard.kicad_sch (KiCad schematic)
At the start: 68 parts, among them J1 IPS114, J2 USB-Type-C, J3 BTB_02x30, J4 BTB_02x30, J5 SH1.0_4P, J6 SH1.0_2P, J7 SH1.0_2P, SW1 3x4, SW2 3x4, SW3 3x4, SW4 3x4, U1 RT9013-33GB, U2 CH343P, U3 SN65HVD232, U4 SN65HVD232, U6 MPU-6050, Y1 32.768KHz, Y2 8MHz

Commit message: 母板pcb初步排布
Parts:
- R1: value (none) -> 10R
- R4, R6: value (none) -> 4.7K
- R5: value (none) -> 10K
- U5: value (none) -> MM32F5277E9P
