File: 1.Hardware/1.FrontCar/2.MotherBoard/Ports.kicad_sch (KiCad schematic)
At the start: 17 parts, among them J10 MOTOR, J11 MOTOR, J12 Maple, J13 SERVO, J14 IO, J15 IO, J16 IO, J17 IO, J18 Conn_02x05_Odd_Even, J2 AUX, J3 PWR, J4 TOF, J5 L_ENCODER, J6 WIRELESS, J7 PWR, J8 R_ENCODER, J9 ELEMAG

Commit message: 母板基本设计完成
Parts:
- removed J7: PWR, Connector:VCC_CONN, symbol Connector_Generic:Conn_01x02
- added PWR: PWR, Connector:VCC_CONN, symbol Connector_Generic:Conn_01x02
Connections:
- net GNDPWR: now also J10.1 (Pin_1), PWR.1 (Pin_1); no longer J10.2 (Pin_2)
- net MOTOR_PWR: now also J10.2 (Pin_2); no longer J10.1 (Pin_1)
- net VBUS: now also PWR.2 (Pin_2)
Changed lines of the file:
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@@
+    )
+  )
+  (symbol (lib_id "Connector_Generic:Conn_01x02") (at 123.19 45.72 0) (mirror x) (unit 1)
+    (in_bom yes) (on_board yes) (dnp no)
+    (property "Reference" "PWR" (at 125.222 45.2847 0)
+      (effects (font (size 1.27 1.27)) (justify left))
+    )
+    (property "Value" "PWR" (at 125.222 42.7478 0)
+      (effects (font (size 1.27 1.27)) (justify left))
+    )
+    (property "Footprint" "Connector_AMASS:AMASS_XT30U-M_1x02_P5.0mm_Vertical" (at 123.19 45.72 0)
+      (effects (font (size 1.27 1.27)) hide)
+    )
+    (property "Datasheet" "" (at 123.19 45.72 0)
+      (effects (font (size 1.27 1.27)) hide)
+    )
+    (property "Datasheet" "" (at 123.19 45.72 0)
+      (effects (font (size 1.27 1.27)) hide)
+    )
+    (property "Footprint" "Connector:VCC_CONN" (at 123.19 45.72 0)
+      (effects (font (size 1.27 1.27)) hide)
+    )
+    (property "Reference" "J?" (at 123.19 45.72 0)
+      (effects (font (size 1.27 1.27)) hide)
+    )
+    (property "Value" "PWR" (at 123.19 45.72 0)
+      (effects (font (size 1.27 1.27)) hide)
+    )
+    (pin "1")
+    (pin "2")
+    (instances
+      (project "FrontCarMotherBoard"
+        (path "/e63e39d7-6ac0-4ffd-8aa3-1841a4541b55/d9d9f6f9-69cc-476c-8327-3871668605e9"
+          (reference "PWR") (unit 1)
+        )
+      )
     )
   )
@@
     )
   )
-  (symbol (lib_id "Connector_Generic:Conn_01x02") (at 123.19 43.18 0) (unit 1)
-    (in_bom yes) (on_board yes) (dnp no)
-    (property "Reference" "J7" (at 125.222 43.6153 0)
-      (effects (font (size 1.27 1.27)) (justify left))
-    )
-    (property "Value" "PWR" (at 125.222 46.1522 0)
-      (effects (font (size 1.27 1.27)) (justify left))
-    )
-    (property "Footprint" "Connector_AMASS:AMASS_XT30U-M_1x02_P5.0mm_Vertical" (at 123.19 43.18 0)
-      (effects (font (size 1.27 1.27)) hide)
-    )
-    (property "Datasheet" "" (at 123.19 43.18 0)
-      (effects (font (size 1.27 1.27)) hide)
-    )
-    (property "Datasheet" "" (at 123.19 43.18 0)
-      (effects (font (size 1.27 1.27)) hide)
-    )
-    (property "Footprint" "Connector:VCC_CONN" (at 123.19 43.18 0)
-      (effects (font (size 1.27 1.27)) hide)
-    )
-    (property "Reference" "J?" (at 123.19 43.18 0)
-      (effects (font (size 1.27 1.27)) hide)
-    )
-    (property "Value" "PWR" (at 123.19 43.18 0)
-      (effects (font (size 1.27 1.27)) hide)
-    )
-    (pin "1")
-    (pin "2")
-    (instances
-      (project "FrontCarMotherBoard"
-        (path "/e63e39d7-6ac0-4ffd-8aa3-1841a4541b55/d9d9f6f9-69cc-476c-8327-3871668605e9"
-          (reference "J7") (unit 1)
+  (symbol (lib_id "Connector_Generic:Conn_01x02") (at 127 61.595 0) (mirror x) (unit 1)
+    (in_bom yes) (on_board yes) (dnp no)
+    (property "Reference" "J10" (at 129.032 61.1597 0)
+      (effects (font (size 1.27 1.27)) (justify left))
+    )
+    (property "Value" "MOTOR" (at 129.032 58.6228 0)
+      (effects (font (size 1.27 1.27)) (justify left))
+    )
+    (property "Footprint" "Connector_AMASS:AMASS_XT30U-M_1x02_P5.0mm_Vertical" (at 127 61.595 0)
+      (effects (font (size 1.27 1.27)) hide)
+    )
+    (property "Datasheet" "~" (at 127 61.595 0)
+      (effects (font (size 1.27 1.27)) hide)
+    )
+    (pin "1")
+    (pin "2")
+    (instances
+      (project "FrontCarMotherBoard"
+        (path "/e63e39d7-6ac0-4ffd-8aa3-1841a4541b55/d9d9f6f9-69cc-476c-8327-3871668605e9"
+          (reference "J10") (unit 1)
         )
       )
@@
         )
       )
-    )
-  )
-  (symbol (lib_id "Connector_Generic:Conn_01x02") (at 127 59.055 0) (unit 1)
-    (in_bom yes) (on_board yes) (dnp no) (fields_autoplaced)
-    (property "Reference" "J10" (at 129.032 59.4903 0)
-      (effects (font (size 1.27 1.27)) (justify left))
-    )
-    (property "Value" "MOTOR" (at 129.032 62.0272 0)
-      (effects (font (size 1.27 1.27)) (justify left))
-    )
-    (property "Footprint" "Connector_AMASS:AMASS_XT30U-M_1x02_P5.0mm_Vertical" (at 127 59.055 0)
-      (effects (font (size 1.27 1.27)) hide)
-    )
-    (property "Datasheet" "~" (at 127 59.055 0)
-      (effects (font (size 1.27 1.27)) hide)
-    )
-    (pin "1")
-    (pin "2")
-    (instances
-      (project "FrontCarMotherBoard"
-        (path "/e63e39d7-6ac0-4ffd-8aa3-1841a4541b55/d9d9f6f9-69cc-476c-8327-3871668605e9"
-          (reference "J10") (unit 1)
-        )
-      )
