File: 1.Hardware/1.CoreBoard/CH32V3_CoreBoard.kicad_pcb (KiCad board)
At the start: 4 copper layers, 38.2 x 25.2 mm, 53 parts, among them J2 SH1.0_4P, J4 BTB_02X18, J5 BTB_02X18, SW1 3x4, SW2 3x4, SW3 3x4, SW4 3x4, U2 RT9013-33GB, U3 BMI270, U5 IPS096, Y1 32.768KHz, Y2 8MHz

Commit message: coreboard
Connections:
- J5 pad 27: /PD10 -> /PB12
- J5 pad 29: /PD8 -> /PE15
- J5 pad 30: /ENC_2DIR -> /PD10
- J5 pad 31: /PB12 -> /PE14
- J5 pad 32: /PB14 -> /ENC_2DIR
- J5 pad 33: /UART7_TX -> /UART7_RX
- J5 pad 34: /UART7_RX -> /PD8
- J5 pad 35: /PE14 -> /UART7_TX
- J5 pad 36: /PE15 -> /PB14
Routing:
- net /CAM_D6: track 0.00 -> 23.3 mm, vias 0 -> 2
- net /CAM_D5: track 0.00 -> 23.3 mm, vias 0 -> 2
- net /CAM_D7: track 0.00 -> 22.5 mm, vias 0 -> 2
- net /CAM_TXD: track 0.00 -> 22.4 mm, vias 0 -> 2
- net /UART3_TX: track 0.00 -> 21.6 mm
- net /UART3_RX: track 0.00 -> 20.9 mm
- net /CAM_RXD: track 0.00 -> 20.0 mm, vias 0 -> 2
- net /CAM_VSYNC: track 0.00 -> 19.2 mm, vias 0 -> 2
- net /CAM_HREF: track 0.00 -> 18.9 mm, vias 0 -> 2
- net /CAM_D4: track 0.00 -> 18.9 mm, vias 0 -> 2
- net /DAP_SWCLK: track 0.00 -> 18.9 mm, vias 0 -> 1
- net /DAP_SWDIO: track 0.00 -> 18.8 mm, vias 0 -> 1
- net /CAM_PLCK: track 0.00 -> 17.1 mm, vias 0 -> 2
- net /PA11: track 0.00 -> 16.8 mm, vias 0 -> 2
- net /CAM_D0: track 0.00 -> 14.8 mm, vias 0 -> 2
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
Commit message: update
Parts:
- moved C10 1.91 mm to (226.3, 104.5), turned to 90 degrees
- moved C11 1.85 mm to (226.3, 102.6), turned to -90 degrees
- turned Y2 to 180 degrees
Routing:
- net /DAP_SWDIO: track 18.8 -> 49.9 mm, vias 1 -> 4
- net /DAP_SWCLK: track 18.9 -> 48.3 mm, vias 1 -> 4
- net /DAP_LED: track 0.00 -> 22.7 mm, vias 0 -> 1
- net /UART3_TX: track 21.6 -> 38.9 mm, vias 0 -> 2
- net /UART3_RX: track 20.9 -> 31.5 mm, vias 0 -> 2
- net /OSC_P: track 1.99 -> 11.4 mm
- net +5V: track 0.00 -> 8.31 mm, vias 0 -> 1
- net /IMU_CS: track 0.00 -> 7.74 mm
- net /OSC_N: track 4.46 -> 11.1 mm
- net /IMU_MISO: track 0.00 -> 5.78 mm, vias 0 -> 2
- net /IMU_MOSI: track 0.00 -> 5.38 mm, vias 0 -> 2
- net +3.3VA: track 0.00 -> 4.07 mm
- net GNDA: track 0.00 -> 3.47 mm
- net /IMU_SCK: track 0.00 -> 3.36 mm, vias 0 -> 2
- net +5VA: track 0.00 -> 3.24 mm
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
Commit message: CoreBoard finished
Parts:
- added C22: 100nF, ErBW_s:C_0402, B.Cu at (223.0, 101.8)
- added G***: LOGO, ErBW_s:ErBW_s_1x1cm, F.Cu at (205.5, 96.1)
- moved C10 0.52 mm to (226.3, 105.0)
- moved C11 0.52 mm to (226.3, 103.1)
- moved Y2 0.52 mm to (223.5, 104.1)
- moved R5 0.43 mm to (198.8, 107.3)
- turned C6 to 0 degrees
Connections:
- J4 pad 1: /AUX_SCL -> /PC3
- J4 pad 10: /ADC_VBAT -> /PA7
- J4 pad 11: /PA3 -> /AUX_SDA
- J4 pad 12: /PA7 -> /PC4
- J4 pad 13: /PC4 -> /AUX_SCL
- J4 pad 15: /PB0 -> /PE1
- J4 pad 16: /PB1 -> /PB0
- J4 pad 17: /PE7 -> /PE0
- J4 pad 18: /PE8 -> /PB1
- J4 pad 19: /PE9 -> /PD6
- J4 pad 2: /AUX_SDA -> /ADC_VBAT
- J4 pad 20: /PE10 -> /PE7
- J4 pad 21: /PE11 -> /PD5
- J4 pad 22: /PE0 -> /PE8
- J4 pad 23: /PE1 -> /ENC_1LSB
- J4 pad 24: /PD5 -> /PE9
- J4 pad 25: /PD6 -> /PD2
- J4 pad 26: /PD2 -> /PE10
- J4 pad 27: /ENC_1LSB -> /ENC_1DIR
- J4 pad 28: /PA15 -> /PE11
- J4 pad 29: /ENC_1DIR -> /PA15
- J4 pad 3: /BUZZER -> /PC2
- J4 pad 4: /PC0 -> /ADC_DIS
- J4 pad 6: /PC2 -> /PA0
- J4 pad 7: /PC3 -> /PC0
- J4 pad 8: /PA0 -> /PA3
- J4 pad 9: /ADC_DIS -> /BUZZER
- U1 pad 2: /ENCODER_B -> /KEY_CENTER
- U1 pad 3: /KEY_CENTER -> /ENCODER_B
Routing:
- net +3.3V: track 11.3 -> 156.9 mm, vias 0 -> 11
- net Net-(D2-K): track 0.00 -> 55.5 mm, vias 0 -> 2
- net /PE11: track 0.00 -> 27.9 mm, vias 0 -> 2
- net /PE10: track 0.00 -> 27.6 mm, vias 0 -> 2
- net /RST: track 0.00 -> 27.2 mm, vias 0 -> 3
- net /PE8: track 0.00 -> 26.9 mm, vias 0 -> 2
- net /PE7: track 0.00 -> 26.5 mm, vias 0 -> 2
- net +5VA: track 3.24 -> 29.2 mm
- net /PE9: track 1.56 -> 27.2 mm, vias 1 -> 2
- net /PB1: track 0.00 -> 25.0 mm, vias 0 -> 2
- net /PB0: track 0.00 -> 24.5 mm, vias 0 -> 2
- net /PC5: track 0.00 -> 23.9 mm, vias 0 -> 2
- net /PC4: track 0.00 -> 23.3 mm, vias 0 -> 2
- net /PA15: track 0.00 -> 23.2 mm, vias 0 -> 2
- net /PA7: track 0.00 -> 22.8 mm, vias 0 -> 2
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- added copper zone on B.Cu, net GND
- added copper zone on F.Cu, net GND
- added copper zone on In1.Cu, net GND
- added copper zone on In2.Cu, net GND
Other:
- board text added: "#CH32V3"
- board text added: "DHU 2023 敏感词汇队"
- board text added: "ErBW_s"
- board text added: "IAP"
- board text added: "JLCJLCJLCJLC"
- board text added: "Link"
- board text added: "PWR"
- board text added: "RST"
- board text added: "SCEP"
- board text added: "Ver1.2 Designed by"
- board text added: "X"
- board text added: "Y"
- board text added: "Z"

Commit message: Fix CoreBoard for production
Other:
- board size 38.2 x 25.2 mm -> 38.3 x 25.2 mm
