File: 1.Hardware/2.MotherBoard/MotherBoard.kicad_pcb (KiCad board)
At the start: 2 copper layers, 68 parts, among them J1 9-Axis, J10 GPS, J4 WIRELESS, J5 MOTOR, J6 FLY_WHEEL, J7 MOTOR, J8 MOTOR_BACK, J9 SERVO, Q1 S8050, SW1 SW_SPDT, U1 ME3116, U2 RT9013-33GB, U3 ME3116, U4 SCEP_CH32V3, U5 MT9V034

Commit message: MotherBoard finished
Parts:
- added REF**: MountingHole_3.2mm_M3_Pad, MountingHole:MountingHole_3.2mm_M3_Pad, F.Cu at (76.4, 3.15)
- added REF**: MountingHole_3.2mm_M3_Pad, MountingHole:MountingHole_3.2mm_M3_Pad, F.Cu at (76.4, 44.2)
- added REF**: MountingHole_3.2mm_M3_Pad, MountingHole:MountingHole_3.2mm_M3_Pad, F.Cu at (29.8, 3.15)
- added REF**: MountingHole_3.2mm_M3_Pad, MountingHole:MountingHole_3.2mm_M3_Pad, F.Cu at (29.8, 44.2)
- C1, C10, C11, C12, C13, C14, C15, C16, C17, C3, C4, C5, C6, C8, C9: footprint Capacitor_SMD:C_0603_1608Metric -> ErBW_s:C_0402
- C7: footprint Capacitor_SMD:C_0603_1608Metric -> ErBW_s:C_0402; moved to F.Cu
- D2, D4, D5: footprint LED_SMD:LED_0805_2012Metric -> LED_SMD:LED_0603_1608Metric
- L1, L2: footprint Inductor_SMD:L_Sunlord_SWPA4030S -> ErBW_s:L_NR201612
- R1, R10, R11, R12, R13, R14, R15, R16, R17, R18, R20, R3, R4, R5, R7, R8, R9, R?: footprint Resistor_SMD:R_0603_1608Metric -> ErBW_s:R_0402
- R19: moved to B.Cu
- R2, R6: footprint Resistor_SMD:R_0603_1608Metric -> ErBW_s:R_0402; moved to F.Cu
- TP1, TP2, TP?: footprint TestPoint:TestPoint_Pad_D1.5mm -> TestPoint:TestPoint_Pad_D1.0mm
- TP4: footprint TestPoint:TestPoint_Pad_1.5x1.5mm -> TestPoint:TestPoint_Pad_1.0x1.0mm
- moved R7 69.5 mm to (62.9, 25.4)
- moved R5 61.1 mm to (62.9, 28.8), turned to 180 degrees
- moved R4 60.8 mm to (62.9, 26.5), turned to 180 degrees
- moved R11 54.8 mm to (77.6, 16.4), turned to 180 degrees
- moved D4 53.6 mm to (77.0, 18.0), turned to 180 degrees
- moved R14 52.9 mm to (45.0, 43.0)
- moved R8 49.6 mm to (62.9, 27.6)
- moved C11 49.6 mm to (75.9, 14.4), turned to -90 degrees
- moved C10 49.1 mm to (77.6, 15.1), turned to 180 degrees
- moved U2 49.1 mm to (77.1, 10.7), turned to -90 degrees
- moved R13 48.4 mm to (45.0, 45.3)
- moved R17 44.4 mm to (45.0, 41.8), turned to 180 degrees
- moved C9 41.2 mm to (77.6, 13.8), turned to 180 degrees
- moved R16 40.4 mm to (45.0, 44.1), turned to 180 degrees
- moved R6 28.6 mm to (62.9, 31.1)
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Connections:
- C7 pad 1: GNDPWR -> GND
- J5 pad 1: GNDPWR -> GND
- J7 pad 1: GNDPWR -> GND
- R6 pad 2: GNDPWR -> GND
Routing:
- net /MOTOR_PWR: track 0.00 -> 121.5 mm
- net +5V: track 0.00 -> 75.8 mm, vias 0 -> 3
- net VCC: track 0.00 -> 60.0 mm, vias 0 -> 2
- net /UART7_TX: track 0.00 -> 51.4 mm, vias 0 -> 1
- net /UART7_RX: track 0.00 -> 50.7 mm, vias 0 -> 1
- net +3V3: track 0.00 -> 49.8 mm, vias 0 -> 3
- net /SERVO: track 0.00 -> 38.0 mm, vias 0 -> 2
- net +6V: track 0.00 -> 37.2 mm
- net /UART8_TX: track 0.00 -> 34.0 mm, vias 0 -> 1
- net /MOTOR_SPD_IN: track 0.00 -> 32.7 mm, vias 0 -> 2
- net /UART8_RX: track 0.00 -> 31.5 mm, vias 0 -> 1
- net /MOTOR_DIR_IN: track 0.00 -> 29.8 mm, vias 0 -> 2
- net /MOTOR_DIR: track 0.00 -> 27.5 mm, vias 0 -> 2
- net /BUZZER: track 0.00 -> 26.4 mm
- net /CAM_PLCK: track 0.00 -> 25.7 mm
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- added copper zone on B.Cu, net GND
- added copper zone on F.Cu, net GND
- added copper zone on B.Cu, net GNDPWR
- added copper zone on F.Cu, net GNDPWR
Other:
- board outline added: 56.7 x 59 mm
- board text added: "3V3"
- board text added: "5V"
- board text added: "6V"
- board text added: "MountingHole_3.2mm_M3_Pad"
- board text added: "东华大学 2023 敏感词汇队"
