File: 1.Hardware/3.BLDC/3.AlO/AIO.kicad_pcb (KiCad board)
At the start: 4 copper layers, 63.1 x 63.5 mm, 154 parts, among them IC1 FD6288Q, IC2 FD6288Q, J1 FLY_WHEEL, J2 SWD&UART, J3 MOTOR_BACK, J4 MR30, J5 MR30, J6 Hall, J7 Hall, J8 MOTOR, J9 MOTOR, Q1 NMOS, Q10 NMOS, Q11 NMOS, Q12 NMOS, Q2 NMOS, Q3 NMOS, Q4 NMOS, Q5 NMOS, Q6 NMOS, Q7 NMOS, Q8 NMOS, Q9 NMOS, SW1 SW_SPDT, SW2 SW_SPDT, U2 RT9013-33GB, U3 ME3116, Y1 8MHz

Commit message: Update AIO pcb
Parts:
- moved R49 7.53 mm to (149.1, 89.0), turned to 0 degrees
- moved R50 7.53 mm to (149.1, 113.2), turned to 0 degrees
- moved D12 0.80 mm to (177.5, 82.5)
Routing:
- net /PWMCH: track 0.00 -> 37.7 mm, vias 0 -> 2
- net /PWMBH: track 0.00 -> 34.9 mm, vias 0 -> 2
- net /PWMAH: track 0.00 -> 34.2 mm, vias 0 -> 2
- net Net-(D2-A): track 12.3 -> 40.5 mm
- net /PWMWL: track 0.00 -> 25.4 mm, vias 0 -> 2
- net /PWMWH: track 0.00 -> 24.8 mm, vias 0 -> 2
- net /PWMVL: track 0.00 -> 24.7 mm, vias 0 -> 2
- net /PWMVH: track 0.00 -> 23.5 mm, vias 0 -> 2
- net /HOA: track 0.00 -> 23.5 mm, vias 0 -> 2
- net /LOA: track 0.00 -> 23.1 mm, vias 0 -> 2
- net /HOB: track 0.00 -> 22.8 mm, vias 0 -> 2
- net /LOW: track 0.00 -> 22.2 mm, vias 0 -> 2
- net /PWMUL: track 0.00 -> 22.1 mm, vias 0 -> 2
- net /PWMUH: track 0.00 -> 22.1 mm, vias 0 -> 2
- net /PWMCL: track 0.00 -> 22.0 mm, vias 0 -> 2
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- added copper zone on B.Cu, net +12V
- added copper zone on F.Cu, net +12V
- added copper zone on F.Cu, net /A
- added copper zone on F.Cu, net /B
- added copper zone on F.Cu, net /C
- added copper zone on B.Cu, net /ISUM1
- added copper zone on F.Cu, net /ISUM1
- added copper zone on B.Cu, net /ISUM2
- added copper zone on F.Cu, net /ISUM2
- added copper zone on F.Cu, net /U
- added copper zone on F.Cu, net /V
- added copper zone on F.Cu, net /W

Commit message: Yet another update of aio driver pcb
Parts:
- added D11: 1N4148W, Diode_SMD:D_SMA, F.Cu at (178.8, 82.3)
- moved D12 2.78 mm to (174.7, 82.3)
Connections:
- J8 pad 1: GND -> unconnected-(J8-Pin_1-Pad1)
- J8 pad 2: +12V -> unconnected-(J8-Pin_2-Pad2)
- J9 pad 2: +12V -> VCC
Routing:
- net +12V: track 3.58 -> 100.9 mm, vias 36 -> 43
- net +5V: track 50.2 -> 102.3 mm
- net /ISUM1: track 0.00 -> 33.1 mm, vias 25 -> 26
- net /ISUM2: track 0.43 -> 18.7 mm
- net VCC: track 0.00 -> 5.83 mm
- net /WHEEL_SPD_OUT: track 36.7 -> 40.1 mm

Commit message: Finished AIO BLDC driver
Parts:
- added REF**: MountingHole_3.2mm_M3_Pad, MountingHole:MountingHole_3.2mm_M3_Pad, F.Cu at (189.6, 68.4)
- added REF**: MountingHole_3.2mm_M3_Pad, MountingHole:MountingHole_3.2mm_M3_Pad, F.Cu at (137.0, 68.4)
Connections:
- C12 pad 2: Net-(IC1-VS2) -> /B
- C13 pad 2: Net-(IC2-VS2) -> /V
- C16 pad 2: Net-(IC1-VS3) -> /C
- C17 pad 2: Net-(IC2-VS3) -> /W
- C3 pad 2: Net-(IC1-VS1) -> /A
- C4 pad 2: Net-(IC2-VS1) -> /U
- IC1 pad 12: Net-(IC1-VS3) -> /C
- IC1 pad 15: Net-(IC1-VS2) -> /B
- IC1 pad 18: Net-(IC1-VS1) -> /A
- IC2 pad 12: Net-(IC2-VS3) -> /W
- IC2 pad 15: Net-(IC2-VS2) -> /V
- IC2 pad 18: Net-(IC2-VS1) -> /U
Routing:
- net +3.3V: track 23.0 -> 133.9 mm, vias 0 -> 8
- net /A: track 0.00 -> 29.7 mm, vias 18 -> 2
- net /W: track 0.00 -> 25.8 mm, vias 17 -> 2
- net /U: track 0.00 -> 23.8 mm, vias 18 -> 2
- net /B: track 0.00 -> 23.7 mm, vias 10 -> 2
- net /V: track 0.00 -> 22.9 mm, vias 8 -> 2
- net /C: track 0.00 -> 21.9 mm, vias 17 -> 2
- net Net-(IC2-VS1): track 3.08 -> 0.00 mm
- net Net-(IC1-VS1): track 3.08 -> 0.00 mm
- net Net-(IC2-VS3): track 2.55 -> 0.00 mm
- net Net-(IC1-VS3): track 2.55 -> 0.00 mm
- net Net-(IC2-VS2): track 2.15 -> 0.00 mm
- net Net-(IC1-VS2): track 2.15 -> 0.00 mm
- net /OP1O: track 28.2 -> 28.9 mm
- net /HOU: track 16.2 -> 16.7 mm
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- added copper zone on B.Cu, net GND
- added copper zone on F.Cu, net GND
- added copper zone on In1.Cu, net GND
- added copper zone on In2.Cu, net GND
Other:
- outline, holes or cut-outs redrawn
- board text added: "OFF"
- board text added: "ON"
- board text added: "东华大学 2023 敏感词汇队"
