File: 1.Hardware/3.BLDC/3.AlO/AIO.kicad_pcb (KiCad board)
At the start: 4 copper layers, 63.1 x 63.5 mm, 157 parts, among them IC1 FD6288Q, IC2 FD6288Q, J1 FLY_WHEEL, J2 SWD&UART, J3 MOTOR_BACK, J4 MR30, J5 MR30, J6 Hall, J7 Hall, J8 MOTOR, J9 MOTOR, Q1 NMOS, Q10 NMOS, Q11 NMOS, Q12 NMOS, Q2 NMOS, Q3 NMOS, Q4 NMOS, Q5 NMOS, Q6 NMOS, Q7 NMOS, Q8 NMOS, Q9 NMOS, SW1 SW_SPDT, SW2 SW_SPDT, U2 RT9013-33GB, U3 ME3116, Y1 8MHz

Commit message: AIO Driver v1.1
Parts:
- moved Q11 7.28 mm to (138.1, 113.2), turned to 180 degrees
- moved Q5 7.28 mm to (145.4, 113.2), turned to -90 degrees
- moved Q1 7.28 mm to (145.4, 80.9), turned to -90 degrees
- moved Q7 7.28 mm to (138.1, 80.9), turned to 180 degrees
- moved Q10 7.28 mm to (138.1, 105.1), turned to 180 degrees
- moved Q12 7.28 mm to (138.1, 121.2), turned to 180 degrees
- moved Q2 7.28 mm to (145.4, 89.0), turned to -90 degrees
- moved Q3 7.28 mm to (145.4, 97.1), turned to -90 degrees
- moved Q4 7.28 mm to (145.4, 105.1), turned to -90 degrees
- moved Q6 7.28 mm to (145.4, 121.2), turned to -90 degrees
- moved Q8 7.28 mm to (138.1, 89.0), turned to 180 degrees
- moved Q9 7.28 mm to (138.1, 97.1), turned to 180 degrees
- moved R21 7.01 mm to (142.8, 84.5)
- moved R23 7.01 mm to (142.8, 100.6)
- moved R24 7.01 mm to (142.8, 108.6)
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Routing:
- net +12V: track 100.9 -> 80.3 mm, vias 43 -> 13
- net /ISUM1: track 33.1 -> 50.7 mm, vias 26 -> 19
- net /ISUM2: track 18.7 -> 28.1 mm, vias 37 -> 19
- net /C: track 21.9 -> 31.0 mm, vias 2 -> 17
- net /LOA: track 23.1 -> 31.6 mm
- net /V: track 22.9 -> 30.7 mm, vias 2 -> 17
- net /B: track 23.7 -> 31.4 mm, vias 2 -> 17
- net /U: track 23.8 -> 31.4 mm, vias 2 -> 17
- net /LOU: track 16.7 -> 23.7 mm
- net /LOV: track 19.9 -> 13.6 mm
- net /W: track 25.8 -> 32.0 mm, vias 2 -> 17
- net /HOW: track 21.1 -> 27.2 mm
- net /HOB: track 23.2 -> 17.9 mm
- net /LOB: track 19.2 -> 23.9 mm
- net /HOV: track 17.3 -> 21.8 mm
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- removed copper zone on B.Cu, net +12V
Other:
- board text added: "AIO BLDC Driver v1.1"
- board text added: "Designed by ErBW_s"
