File: 1.Hardware/3.BLDC/3.AlO/AIO.kicad_sch (KiCad schematic)
At the start: 154 parts, among them IC1 FD6288Q, IC2 FD6288Q, J1 FLY_WHEEL, J2 MOTOR, J3 MOTOR_BACK, J3 MR30, J4 MOTOR, J4 MR30, J5 Hall, J7 Hall, J8 SWD&UART, Q1 NMOS, Q10 NMOS, Q11 NMOS, Q12 NMOS, Q2 NMOS, Q3 NMOS, Q4 NMOS, Q5 NMOS, Q6 NMOS, Q7 NMOS, Q8 NMOS, Q9 NMOS, SW1 SW_SPDT, SW2 SW_SPDT, U3 ME3116, U4 RT9013-33GB, Y1 8MHz

Commit message: 摆烂AIO
Parts:
- D1, D3: footprint ErBW_s:LED_0402 -> LED_SMD:LED_0603_1608Metric
- D11: footprint Diode_SMD:D_SOD-323 -> Diode_SMD:D_SMB
- J5, J7: footprint (none) -> Connector_JST:JST_ZE_SM06B-ZESS-TB_1x06-1MP_P1.50mm_Horizontal
- J8: footprint (none) -> Connector_JST:JST_SH_SM05B-SRSS-TB_1x05-1MP_P1.00mm_Horizontal
- SW1, SW2: footprint (none) -> ErBW_s:SPDT_12C01
Connections:
- net CU_SUM1: no longer R27.1
- net CU_SUM2: no longer R27.1
- net OP1O: now also R27.1
- net OP3O: now also R27.1
Changed lines of the file:
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@@
   (junction (at 86.995 241.3) (diameter 0) (color 0 0 0 0)
   )
+  (junction (at 189.865 93.345) (diameter 0) (color 0 0 0 0)
+  )
   (junction (at 164.465 132.715) (diameter 0) (color 0 0 0 0)
   )
@@
   (junction (at 113.665 195.58) (diameter 0) (color 0 0 0 0)
   )
+  (junction (at 190.5 52.705) (diameter 0) (color 0 0 0 0)
+  )
   (junction (at 368.935 145.415) (diameter 0) (color 0 0 0 0)
   )
@@
     (stroke (width 0) (type default))
   )
-  (wire (pts (xy 200.025 35.56) (xy 200.025 52.705))
-    (stroke (width 0) (type default))
-  )
   (wire (pts (xy 283.845 181.61) (xy 283.845 177.165))
     (stroke (width 0) (type default))
@@
     (stroke (width 0) (type default))
   )
-  (wire (pts (xy 184.785 52.705) (xy 193.04 52.705))
+  (wire (pts (xy 184.785 52.705) (xy 190.5 52.705))
     (stroke (width 0) (type default))
   )
@@
     (stroke (width 0) (type default))
   )
-  (wire (pts (xy 182.245 76.2) (xy 199.39 76.2))
+  (wire (pts (xy 182.245 76.2) (xy 189.865 76.2))
     (stroke (width 0) (type default))
   )
@@
     (stroke (width 0) (type default))
   )
+  (wire (pts (xy 189.865 76.2) (xy 189.865 93.345))
+    (stroke (width 0) (type default))
+  )
   (wire (pts (xy 80.645 130.81) (xy 80.645 129.54))
     (stroke (width 0) (type default))
@@
     (stroke (width 0) (type default))
   )
+  (wire (pts (xy 190.5 35.56) (xy 190.5 52.705))
+    (stroke (width 0) (type default))
+  )
+  (wire (pts (xy 189.865 93.345) (xy 192.405 93.345))
+    (stroke (width 0) (type default))
+  )
   (wire (pts (xy 37.465 198.12) (xy 35.56 198.12))
     (stroke (width 0) (type default))
@@
     (stroke (width 0) (type default))
   )
-  (wire (pts (xy 199.39 76.2) (xy 199.39 93.345))
-    (stroke (width 0) (type default))
-  )
   (wire (pts (xy 54.61 198.12) (xy 66.675 198.12))
     (stroke (width 0) (type default))
@@
     (stroke (width 0) (type default))
   )
-  (wire (pts (xy 184.15 93.345) (xy 192.405 93.345))
+  (wire (pts (xy 184.15 93.345) (xy 189.865 93.345))
     (stroke (width 0) (type default))
   )
@@
     (stroke (width 0) (type default))
   )
-  (wire (pts (xy 182.88 35.56) (xy 200.025 35.56))
+  (wire (pts (xy 182.88 35.56) (xy 190.5 35.56))
     (stroke (width 0) (type default))
   )
@@
     (stroke (width 0) (type default))
   )
+  (wire (pts (xy 190.5 52.705) (xy 193.04 52.705))
+    (stroke (width 0) (type default))
+  )
   (wire (pts (xy 37.465 161.925) (xy 38.735 161.925))
     (stroke (width 0) (type default))
@@
       (effects (font (size 1.27 1.27)) (justify right))
     )
-    (property "Footprint" "ErBW_s:LED_0402" (at 97.155 257.81 0)
+    (property "Footprint" "LED_SMD:LED_0603_1608Metric" (at 97.155 257.81 0)
       (effects (font (size 1.27 1.27)) hide)
     )
@@
       (effects (font (size 1.27 1.27)))
     )
-    (property "Footprint" "" (at 289.56 93.345 0)
+    (property "Footprint" "ErBW_s:SPDT_12C01" (at 289.56 93.345 0)
       (effects (font (size 1.27 1.27)) hide)
     )
@@
       (effects (font (size 1.27 1.27)) (justify right))
     )
-    (property "Footprint" "Diode_SMD:D_SOD-323" (at 69.215 217.805 0)
+    (property "Footprint" "Diode_SMD:D_SMB" (at 69.215 217.805 0)
       (effects (font (size 1.27 1.27)) hide)
     )
@@
       (effects (font (size 1.27 1.27)) (justify right))
     )
-    (property "Footprint" "ErBW_s:LED_0402" (at 163.195 257.81 0)
+    (property "Footprint" "LED_SMD:LED_0603_1608Metric" (at 163.195 257.81 0)
       (effects (font (size 1.27 1.27)) hide)
     )
@@
       (effects (font (size 1.27 1.27)))
     )
-    (property "Footprint" "" (at 290.195 52.705 0)
+    (property "Footprint" "ErBW_s:SPDT_12C01" (at 290.195 52.705 0)
       (effects (font (size 1.27 1.27)) hide)
     )
@@
       (effects (font (size 1.27 1.27)) (justify left))
     )
-    (property "Footprint" "" (at 285.115 213.995 0)
+    (property "Footprint" "Connector_JST:JST_ZE_SM06B-ZESS-TB_1x06-1MP_P1.50mm_Horizontal" (at 285.115 213.995 0)
       (effects (font (size 1.27 1.27)) hide)
     )
@@
       (effects (font (size 1.27 1.27)) (justify left))
     )
-    (property "Footprint" "" (at 91.44 186.69 0)
+    (property "Footprint" "Connector_JST:JST_SH_SM05B-SRSS-TB_1x05-1MP_P1.00mm_Horizontal" (at 91.44 186.69 0)
       (effects (font (size 1.27 1.27)) hide)
     )
@@
       (effects (font (size 1.27 1.27)) (justify left))
     )
-    (property "Footprint" "" (at 222.885 213.995 0)
+    (property "Footprint" "Connector_JST:JST_ZE_SM06B-ZESS-TB_1x06-1MP_P1.50mm_Horizontal" (at 222.885 213.995 0)
       (effects (font (size 1.27 1.27)) hide)
     )

Commit message: Yet another update of aio driver pcb
Parts:
- added D1: 1N4148W, Diode_SMD:D_SMA, symbol Diode:1N4148W
Connections:
- net +12V: now also D1.1 (K); no longer J2.2 (Pin_2), J4.2 (Pin_2)
- net GND: no longer J2.1 (Pin_1)
- new net VCC: D1.2 (A), J4.2 (Pin_2)
- no-connect marks 33 -> 35
Changed lines of the file:
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@@
   (junction (at 195.58 216.535) (diameter 0) (color 0 0 0 0)
   )
+  (junction (at 64.135 212.09) (diameter 0) (color 0 0 0 0)
+  )
   (junction (at 504.825 163.195) (diameter 0) (color 0 0 0 0)
   )
@@
   (junction (at 81.28 194.31) (diameter 0) (color 0 0 0 0)
   )
+  (no_connect (at 31.75 212.09))
   (no_connect (at 38.735 62.23))
   (no_connect (at 93.345 121.92))
@@
   (no_connect (at 62.865 121.92))
   (no_connect (at 98.425 34.29))
+  (no_connect (at 31.75 214.63))
   (no_connect (at 103.505 121.92))
   (no_connect (at 62.865 34.29))
@@
     (stroke (width 0) (type default))
   )
-  (wire (pts (xy 30.48 214.63) (xy 31.75 214.63))
-    (stroke (width 0) (type default))
-  )
   (wire (pts (xy 260.35 198.755) (xy 257.81 198.755))
     (stroke (width 0) (type default))
@@
     (stroke (width 0) (type default))
   )
+  (wire (pts (xy 54.61 212.09) (xy 55.245 212.09))
+    (stroke (width 0) (type default))
+  )
   (wire (pts (xy 189.865 93.345) (xy 192.405 93.345))
     (stroke (width 0) (type default))
@@
     (stroke (width 0) (type default))
   )
+  (wire (pts (xy 62.865 212.09) (xy 64.135 212.09))
+    (stroke (width 0) (type default))
+  )
   (wire (pts (xy 525.145 145.415) (xy 530.86 145.415))
     (stroke (width 0) (type default))
@@
     (stroke (width 0) (type default))
   )
+  (wire (pts (xy 65.405 212.09) (xy 64.135 212.09))
+    (stroke (width 0) (type default))
+  )
   (wire (pts (xy 537.21 163.195) (xy 538.48 163.195))
     (stroke (width 0) (type default))
@@
     )
   )
-  (symbol (lib_id "power:GND") (at 30.48 214.63 270) (unit 1)
-    (in_bom yes) (on_board yes) (dnp no)
-    (property "Reference" "#PWR03" (at 24.13 214.63 0)
-      (effects (font (size 1.27 1.27)) hide)
-    )
-    (property "Value" "GND" (at 27.305 214.63 90)
-      (effects (font (size 1.27 1.27)) (justify right))
-    )
-    (property "Footprint" "" (at 30.48 214.63 0)
-      (effects (font (size 1.27 1.27)) hide)
-    )
-    (property "Datasheet" "" (at 30.48 214.63 0)
-      (effects (font (size 1.27 1.27)) hide)
-    )
-    (pin "1")
-    (instances
-      (project "Driver"
-        (path "/28189786-bde1-4400-8acc-7a3b1594a742"
-          (reference "#PWR03") (unit 1)
-        )
-      )
-      (project "MotherBoard"
-        (path "/9bf74166-fa0b-45a3-b1a9-21dd6c95e555"
-          (reference "#PWR07") (unit 1)
-        )
-      )
-      (project "AIO"
-        (path "/cb89e9d5-9241-463a-ab3e-e84174bcfc12"
-          (reference "#PWR058") (unit 1)
-        )
-      )
-      (project "FrontCarMotherBoard"
-        (path "/e63e39d7-6ac0-4ffd-8aa3-1841a4541b55/d9d9f6f9-69cc-476c-8327-3871668605e9"
-          (reference "#PWR?") (unit 1)
-        )
-      )
-    )
-  )
   (symbol (lib_id "power:GND") (at 100.33 213.995 90) (unit 1)
     (in_bom yes) (on_board yes) (dnp no) (fields_autoplaced)
@@
     )
   )
-  (symbol (lib_id "power:+12V") (at 64.135 212.09 0) (unit 1)
+  (symbol (lib_id "power:+12V") (at 65.405 212.09 270) (unit 1)
     (in_bom yes) (on_board yes) (dnp no) (fields_autoplaced)
-    (property "Reference" "#PWR016" (at 64.135 215.9 0)
+    (property "Reference" "#PWR016" (at 61.595 212.09 0)
       (effects (font (size 1.27 1.27)) hide)
     )
-    (property "Value" "+12V" (at 64.135 208.5881 0)
-      (effects (font (size 1.27 1.27)))
+    (property "Value" "+12V" (at 68.58 212.4068 90)
+      (effects (font (size 1.27 1.27)) (justify left))
     )
-    (property "Footprint" "" (at 64.135 212.09 0)
+    (property "Footprint" "" (at 65.405 212.09 0)
       (effects (font (size 1.27 1.27)) hide)
     )
-    (property "Datasheet" "" (at 64.135 212.09 0)
+    (property "Datasheet" "" (at 65.405 212.09 0)
       (effects (font (size 1.27 1.27)) hide)
     )
@@
     )
   )
+  (symbol (lib_id "Diode:1N4148W") (at 59.055 212.09 180) (unit 1)
+    (in_bom yes) (on_board yes) (dnp no) (fields_autoplaced)
+    (property "Reference" "D1" (at 59.055 207.8101 0)
+      (effects (font (size 1.27 1.27)))
+    )
+    (property "Value" "1N4148W" (at 59.055 209.7311 0)
+      (effects (font (size 1.27 1.27)))
+    )
+    (property "Footprint" "Diode_SMD:D_SMA" (at 59.055 207.645 0)
+      (effects (font (size 1.27 1.27)) hide)
+    )
+    (property "Datasheet" "https://www.vishay.com/docs/85748/1n4148w.pdf" (at 59.055 212.09 0)
+      (effects (font (size 1.27 1.27)) hide)
+    )
+    (property "Sim.Device" "D" (at 59.055 212.09 0)
+      (effects (font (size 1.27 1.27)) hide)
+    )
+    (property "Sim.Pins" "1=K 2=A" (at 59.055 212.09 0)
+      (effects (font (size 1.27 1.27)) hide)
+    )
+    (pin "1")
+    (pin "2")
+    (instances
+      (project "MotherBoard"
+        (path "/9bf74166-fa0b-45a3-b1a9-21dd6c95e555"
+          (reference "D1") (unit 1)
+        )
+      )
+      (project "AIO"
+        (path "/cb89e9d5-9241-463a-ab3e-e84174bcfc12"
+          (reference "D11") (unit 1)
+        )
+      )
+      (project "FrontCarMotherBoard"
+        (path "/e63e39d7-6ac0-4ffd-8aa3-1841a4541b55/b6c42b83-27cb-41a6-82a4-0cfe59a023a6"
+          (reference "D?") (unit 1)
+        )
+      )
+    )
+  )
   (symbol (lib_id "Device:R_Small") (at 429.895 145.415 90) (unit 1)
     (in_bom yes) (on_board yes) (dnp no)
@@
     )
   )
+  (symbol (lib_id "power:VCC") (at 54.61 212.09 90) (unit 1)
+    (in_bom yes) (on_board yes) (dnp no) (fields_autoplaced)
+    (property "Reference" "#PWR055" (at 58.42 212.09 0)
+      (effects (font (size 1.27 1.27)) hide)
+    )
+    (property "Value" "VCC" (at 51.435 212.4068 90)
+      (effects (font (size 1.27 1.27)) (justify left))
+    )
+    (property "Footprint" "" (at 54.61 212.09 0)
+      (effects (font (size 1.27 1.27)) hide)
+    )
+    (property "Datasheet" "" (at 54.61 212.09 0)
+      (effects (font (size 1.27 1.27)) hide)
+    )
+    (pin "1")
+    (instances
+      (project "AIO"
+        (path "/cb89e9d5-9241-463a-ab3e-e84174bcfc12"
+          (reference "#PWR055") (unit 1)
+        )
+      )
+    )
+  )
   (symbol (lib_id "Device:C_Small") (at 141.605 254 0) (unit 1)
     (in_bom yes) (on_board yes) (dnp no) (fields_autoplaced)
@@
     )
   )
+  (symbol (lib_id "power:VCC") (at 31.75 224.79 90) (unit 1)
+    (in_bom yes) (on_board yes) (dnp no) (fields_autoplaced)
+    (property "Reference" "#PWR058" (at 35.56 224.79 0)
+      (effects (font (size 1.27 1.27)) hide)
+    )
+    (property "Value" "VCC" (at 28.575 225.1068 90)
+      (effects (font (size 1.27 1.27)) (justify left))
+    )
+    (property "Footprint" "" (at 31.75 224.79 0)
+      (effects (font (size 1.27 1.27)) hide)
+    )
+    (property "Datasheet" "" (at 31.75 224.79 0)
+      (effects (font (size 1.27 1.27)) hide)
+    )
+    (pin "1")
+    (instances
+      (project "AIO"
+        (path "/cb89e9d5-9241-463a-ab3e-e84174bcfc12"
+          (reference "#PWR058") (unit 1)
+        )
+      )
+    )
+  )
   (symbol (lib_id "power:GNDA") (at 36.195 95.25 270) (unit 1)
     (in_bom yes) (on_board yes) (dnp no) (fields_autoplaced)
@@
     )
   )
-  (symbol (lib_id "power:+12V") (at 31.75 224.79 0) (unit 1)
-    (in_bom yes) (on_board yes) (dnp no) (fields_autoplaced)
-    (property "Reference" "#PWR08" (at 31.75 228.6 0)
-      (effects (font (size 1.27 1.27)) hide)
-    )
-    (property "Value" "+12V" (at 31.75 221.2881 0)
-      (effects (font (size 1.27 1.27)))
-    )
-    (property "Footprint" "" (at 31.75 224.79 0)
-      (effects (font (size 1.27 1.27)) hide)
-    )
-    (property "Datasheet" "" (at 31.75 224.79 0)
-      (effects (font (size 1.27 1.27)) hide)
-    )
-    (pin "1")
-    (instances
-      (project "Driver"
-        (path "/28189786-bde1-4400-8acc-7a3b1594a742"
-          (reference "#PWR08") (unit 1)
-        )
-      )
-      (project "AIO"
-        (path "/cb89e9d5-9241-463a-ab3e-e84174bcfc12"
-          (reference "#PWR063") (unit 1)
-        )
-      )
-    )
-  )
   (symbol (lib_id "power:GND") (at 158.75 50.165 270) (unit 1)
     (in_bom yes) (on_board yes) (dnp no)
@@
         )
       )
-    )
-  )
-  (symbol (lib_id "power:+12V") (at 31.75 212.09 0) (unit 1)
-    (in_bom yes) (on_board yes) (dnp no) (fields_autoplaced)
-    (property "Reference" "#PWR07" (at 31.75 215.9 0)
-      (effects (font (size 1.27 1.27)) hide)
-    )
-    (property "Value" "+12V" (at 31.75 208.5881 0)
-      (effects (font (size 1.27 1.27)))
-    )
-    (property "Footprint" "" (at 31.75 212.09 0)
-      (effects (font (size 1.27 1.27)) hide)
-    )
-    (property "Datasheet" "" (at 31.75 212.09 0)
-      (effects (font (size 1.27 1.27)) hide)
-    )
-    (pin "1")
-    (instances
-      (project "Driver"
-        (path "/28189786-bde1-4400-8acc-7a3b1594a742"
-          (reference "#PWR07") (unit 1)
-        )
-      )
-      (project "AIO"
-        (path "/cb89e9d5-9241-463a-ab3e-e84174bcfc12"
-          (reference "#PWR055") (unit 1)
-        )
-      )

Commit message: Finished AIO BLDC driver
Connections:
- net A: now also C11.2, IC1.18 (VS1)
- net B: now also C12.2, IC1.15 (VS2)
- net C: now also C13.2, IC1.12 (VS3)
- net U: now also C28.2, IC2.18 (VS1)
- net V: now also C29.2, IC2.15 (VS2)
- net W: now also C31.2, IC2.12 (VS3)
Changed lines of the file:
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@@
     (effects (font (size 1.27 1.27)) (justify right bottom))
+  )
+  (label "V" (at 297.815 160.655 0) (fields_autoplaced)
+    (effects (font (size 1.27 1.27)) (justify left bottom))
   )
   (label "PWMBH" (at 139.065 64.77 180) (fields_autoplaced)
@@
     (effects (font (size 1.27 1.27)) (justify left bottom))
   )
+  (label "C" (at 197.485 179.07 0) (fields_autoplaced)
+    (effects (font (size 1.27 1.27)) (justify left bottom))
+  )
   (label "BREAK2" (at 271.78 93.345 180) (fields_autoplaced)
     (effects (font (size 1.27 1.27)) (justify right bottom))
@@
     (effects (font (size 1.27 1.27)) (justify left bottom))
   )
+  (label "W" (at 286.385 179.07 0) (fields_autoplaced)
+    (effects (font (size 1.27 1.27)) (justify left bottom))
+  )
   (label "ENC_B" (at 187.325 213.995 0) (fields_autoplaced)
     (effects (font (size 1.27 1.27)) (justify left bottom))
@@
     (effects (font (size 1.27 1.27)) (justify right bottom))
   )
+  (label "B" (at 208.915 160.655 0) (fields_autoplaced)
+    (effects (font (size 1.27 1.27)) (justify left bottom))
+  )
   (label "OP1N" (at 173.355 50.165 0) (fields_autoplaced)
     (effects (font (size 1.27 1.27)) (justify left bottom))
@@
     (effects (font (size 1.27 1.27)) (justify left bottom))
   )
+  (label "U" (at 297.815 153.035 0) (fields_autoplaced)
+    (effects (font (size 1.27 1.27)) (justify left bottom))
+  )
   (label "MOTOR_DIR_OUT" (at 66.675 180.34 180) (fields_autoplaced)
     (effects (font (size 1.27 1.27)) (justify right bottom))
@@
     (effects (font (size 1.27 1.27)) (justify right bottom))
   )
+  (label "A" (at 208.915 153.035 0) (fields_autoplaced)
+    (effects (font (size 1.27 1.27)) (justify left bottom))
+  )
   (label "B" (at 389.255 154.305 0) (fields_autoplaced)

Commit message: Update 3D model to v1.2
Parts:
- Q1, Q10, Q11, Q12, Q2, Q3, Q4, Q5, Q6, Q7, Q8, Q9: symbol Transistor_FET:AO3400A -> ErBW_s:NMOS
Connections:
- net +12V: now also Q1.D, Q3.D, Q5.D, Q7.D, Q8.D, Q9.D; no longer Q1.3 (D), Q3.3 (D), Q5.3 (D), Q7.3 (D), Q8.3 (D), Q9.3 (D)
- net +3.3V: now also R11.1, R12.1, R13.1, R59.1, R60.1, R61.1
- net +5V: no longer R11.1, R12.1, R13.1, R59.1, R60.1, R61.1
- net A: now also Q1.S, Q2.D; no longer Q1.2 (S), Q2.3 (D)
- net B: now also Q3.S, Q4.D; no longer Q3.2 (S), Q4.3 (D)
- net C: now also Q5.S, Q6.D; no longer Q5.2 (S), Q6.3 (D)
- net ISUM1: now also Q2.S, Q4.S, Q6.S; no longer Q2.2 (S), Q4.2 (S), Q6.2 (S)
- net ISUM2: now also Q10.S, Q11.S, Q12.S; no longer Q10.2 (S), Q11.2 (S), Q12.2 (S)
- net U: now also Q10.D, Q7.S; no longer Q10.3 (D), Q7.2 (S)
- net V: now also Q11.D, Q8.S; no longer Q11.3 (D), Q8.2 (S)
- net W: now also Q12.D, Q9.S; no longer Q12.3 (D), Q9.2 (S)
- net at R6.1, R6.2: now also Q9.G; no longer Q9.1 (G)
- net at R6.1, R6.2: now also Q8.G; no longer Q8.1 (G)
- net at R6.1, R6.2: now also Q10.G; no longer Q10.1 (G)
- net at R6.1, R6.2: now also Q12.G; no longer Q12.1 (G)
- net at R6.1, R6.2: now also Q11.G; no longer Q11.1 (G)
- net at R6.1, R6.2: now also Q3.G; no longer Q3.1 (G)
- net at R6.1, R6.2: now also Q1.G; no longer Q1.1 (G)
- net at R6.1, R6.2: now also Q2.G; no longer Q2.1 (G)
- net at R6.1, R6.2: now also Q7.G; no longer Q7.1 (G)
- net at R6.1, R6.2: now also Q6.G; no longer Q6.1 (G)
- net at R6.1, R6.2: now also Q4.G; no longer Q4.1 (G)
- net at R6.1, R6.2: now also Q5.G; no longer Q5.1 (G)
